File: hardware/teensy/teensy.kicad_pcb (KiCad board)
At the start: 2 copper layers, 1 part, among them U1 Teensy3.5

Commit message: still learning kicad
Parts:
- added J1: CONN_16, Connectors:1X16, F.Cu at (97.2, 123.9)
- added R1: 33OHM-0603-1_10W-1%, Resistors:AXIAL-0.3, F.Cu at (176.5, 115.2)

Commit message: added more to sch
Parts:
- added J2: CONN_16, Connectors:1X16, F.Cu at (192.9, 18.2)
- added R10: 33OHM-0603-1_10W-1%, Resistors:AXIAL-0.3, F.Cu at (117.8, 56.8)
- added R11: 33OHM-0603-1_10W-1%, Resistors:AXIAL-0.3, F.Cu at (128.3, 56.8)
- added R12: 33OHM-0603-1_10W-1%, Resistors:AXIAL-0.3, F.Cu at (117.8, 59.7)
- added R13: 33OHM-0603-1_10W-1%, Resistors:AXIAL-0.3, F.Cu at (117.8, 54.0)
- added R14: 33OHM-0603-1_10W-1%, Resistors:AXIAL-0.3, F.Cu at (117.8, 51.1)
- added R15: 33OHM-0603-1_10W-1%, Resistors:AXIAL-0.3, F.Cu at (138.8, 54.0)
- added R16: 33OHM-0603-1_10W-1%, Resistors:AXIAL-0.3, F.Cu at (136.3, 27.8)
- added R17: 390KOHM-0603-1_10W-1%, Resistors:AXIAL-0.3, F.Cu at (138.8, 59.7)
- added R18: 390KOHM-0603-1_10W-1%, Resistors:AXIAL-0.3, F.Cu at (138.8, 56.8)
- added R2: 33OHM-0603-1_10W-1%, Resistors:AXIAL-0.3, F.Cu at (128.3, 54.0)
- added R3: 33OHM-0603-1_10W-1%, Resistors:AXIAL-0.3, F.Cu at (117.8, 62.6)
- added R4: 33OHM-0603-1_10W-1%, Resistors:AXIAL-0.3, F.Cu at (149.2, 56.8)
- added R5: 33OHM-0603-1_10W-1%, Resistors:AXIAL-0.3, F.Cu at (128.3, 51.1)
- added R6: 33OHM-0603-1_10W-1%, Resistors:AXIAL-0.3, F.Cu at (138.8, 51.1)
- added R7: 33OHM-0603-1_10W-1%, Resistors:AXIAL-0.3, F.Cu at (128.3, 62.6)
- added R8: 33OHM-0603-1_10W-1%, Resistors:AXIAL-0.3, F.Cu at (149.2, 54.0)
- added R9: 33OHM-0603-1_10W-1%, Resistors:AXIAL-0.3, F.Cu at (128.3, 59.7)
- moved J1 177.4 mm to (239.7, 18.2), turned to 180 degrees
Connections:
- J1 pad 1: Net-(J1-Pad1) -> /ct9
- J1 pad 11: Net-(J1-Pad11) -> /ct14
- J1 pad 12: Net-(J1-Pad12) -> Net-(J1-Pad10)
- J1 pad 13: Net-(J1-Pad13) -> /ct15
- J1 pad 14: Net-(J1-Pad14) -> Net-(J1-Pad10)
- J1 pad 15: Net-(J1-Pad15) -> /ct16
- J1 pad 16: Net-(J1-Pad16) -> Net-(J1-Pad10)
- J1 pad 2: Net-(J1-Pad2) -> Net-(J1-Pad10)
- J1 pad 3: Net-(J1-Pad3) -> /ct10
- J1 pad 4: Net-(J1-Pad4) -> Net-(J1-Pad10)
- J1 pad 5: Net-(J1-Pad5) -> /ct11
- J1 pad 6: Net-(J1-Pad6) -> Net-(J1-Pad10)
- J1 pad 7: Net-(J1-Pad7) -> /ct12
- J1 pad 8: Net-(J1-Pad8) -> Net-(J1-Pad10)
- J1 pad 9: Net-(J1-Pad9) -> /ct13
- U1 pad 23: Net-(U1-Pad23) -> /ct10
- U1 pad 24: Net-(U1-Pad24) -> /ct11
- U1 pad 30: Net-(U1-Pad30) -> /ct8
- U1 pad 32: Net-(U1-Pad32) -> /ct12
- U1 pad 33: Net-(U1-Pad33) -> /ct13
- U1 pad 34: Net-(U1-Pad34) -> /ct14
- U1 pad 35: Net-(U1-Pad35) -> /ct15
- U1 pad 36: Net-(U1-Pad36) -> /ct16
- U1 pad 41: Net-(U1-Pad41) -> /ct1
- U1 pad 42: Net-(U1-Pad42) -> /ct2
- U1 pad 43: Net-(U1-Pad43) -> /ct9
- U1 pad 44: Net-(U1-Pad44) -> /ct3
- U1 pad 45: Net-(U1-Pad45) -> /ct4
- U1 pad 46: Net-(U1-Pad46) -> /ct5
- U1 pad 47: Net-(U1-Pad47) -> /ct6
- U1 pad 50: Net-(U1-Pad50) -> /ct7

Commit message: more wiring
Parts:
- R1, R10, R11, R12, R13, R14, R15, R16, R2, R3, R4, R5, R6, R7, R8, R9: value 33OHM-0603-1_10W-1% -> RESISTORAXIAL-0.3
- R17, R18: value 390KOHM-0603-1_10W-1% -> RESISTORAXIAL-0.3
- moved R12 125.2 mm to (239.6, 31.2), turned to 90 degrees
- moved R3 111.3 mm to (224.6, 31.3), turned to 90 degrees
- moved R10 105.4 mm to (220.0, 31.2), turned to 90 degrees
- moved R11 104.5 mm to (229.6, 31.3), turned to 90 degrees
- moved R4 89.3 mm to (234.8, 31.4), turned to 90 degrees
- moved R2 89.0 mm to (214.5, 31.7), turned to 90 degrees
- moved R1 88.0 mm to (204.4, 31.8), turned to 90 degrees
- moved R9 85.6 mm to (209.2, 31.6), turned to 90 degrees
- moved R7 58.5 mm to (178.1, 31.9), turned to 90 degrees
- moved R14 58.0 mm to (172.5, 32.0), turned to 90 degrees
- moved R16 57.0 mm to (193.1, 32.0), turned to 90 degrees
- moved R13 50.6 mm to (163.2, 31.6), turned to 90 degrees
- moved R15 49.2 mm to (182.7, 31.8), turned to 90 degrees
- moved R8 44.6 mm to (187.9, 31.8), turned to 90 degrees
- moved R5 35.3 mm to (157.5, 31.4), turned to 90 degrees
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Connections:
- J1 pad 10: Net-(J1-Pad10) -> /CT_BIAS
- J1 pad 12: Net-(J1-Pad10) -> /CT_BIAS
- J1 pad 14: Net-(J1-Pad10) -> /CT_BIAS
- J1 pad 16: Net-(J1-Pad10) -> /CT_BIAS
- J1 pad 2: Net-(J1-Pad10) -> /CT_BIAS
- J1 pad 4: Net-(J1-Pad10) -> /CT_BIAS
- J1 pad 6: Net-(J1-Pad10) -> /CT_BIAS
- J1 pad 8: Net-(J1-Pad10) -> /CT_BIAS
- J2 pad 10: Net-(J1-Pad10) -> /CT_BIAS
- J2 pad 12: Net-(J1-Pad10) -> /CT_BIAS
- J2 pad 14: Net-(J1-Pad10) -> /CT_BIAS
- J2 pad 16: Net-(J1-Pad10) -> /CT_BIAS
- J2 pad 2: Net-(J1-Pad10) -> /CT_BIAS
- J2 pad 4: Net-(J1-Pad10) -> /CT_BIAS
- J2 pad 6: Net-(J1-Pad10) -> /CT_BIAS
- J2 pad 8: Net-(J1-Pad10) -> /CT_BIAS
- R1 pad P$1: (no net) -> /CT_BIAS
- R1 pad P$2: (no net) -> /ct16
- R10 pad P$1: (no net) -> /CT_BIAS
- R10 pad P$2: (no net) -> /ct13
- R11 pad P$1: (no net) -> /CT_BIAS
- R11 pad P$2: (no net) -> /ct11
- R12 pad P$1: (no net) -> /CT_BIAS
- R12 pad P$2: (no net) -> /ct9
- R13 pad P$1: (no net) -> /CT_BIAS
- R13 pad P$2: (no net) -> /ct7
- R14 pad P$1: (no net) -> /CT_BIAS
- R14 pad P$2: (no net) -> /ct5
- R15 pad P$1: (no net) -> /CT_BIAS
- R15 pad P$2: (no net) -> /ct3
- R16 pad P$1: (no net) -> /CT_BIAS
- R16 pad P$2: (no net) -> /ct1
- R17 pad P$1: (no net) -> /3.3V
- R17 pad P$2: (no net) -> /CT_BIAS
- R18 pad P$1: (no net) -> /CT_BIAS
- R18 pad P$2: (no net) -> /GND
- R2 pad P$1: (no net) -> /CT_BIAS
- R2 pad P$2: (no net) -> /ct14
- R3 pad P$1: (no net) -> /CT_BIAS
- R3 pad P$2: (no net) -> /ct12
- R4 pad P$1: (no net) -> /CT_BIAS
- R4 pad P$2: (no net) -> /ct10
- R5 pad P$1: (no net) -> /CT_BIAS
- R5 pad P$2: (no net) -> /ct8
- R6 pad P$1: (no net) -> /CT_BIAS
- R6 pad P$2: (no net) -> /ct6
- R7 pad P$1: (no net) -> /CT_BIAS
- R7 pad P$2: (no net) -> /ct4
- R8 pad P$1: (no net) -> /CT_BIAS
- R8 pad P$2: (no net) -> /ct2
- R9 pad P$1: (no net) -> /CT_BIAS
- R9 pad P$2: (no net) -> /ct15
- U1 pad 3: Net-(U1-Pad2) -> Net-(U1-Pad3)
- U1 pad 39: Net-(R18-Pad2) -> /GND
- U1 pad 51: Net-(R17-Pad1) -> /3.3V
Routing:
- net /CT_BIAS: track 0.00 -> 115.6 mm

Commit message: fully routed
ugly, but correct, i think.
Parts:
- added J3: CONN_04, Connectors:1X04, F.Cu at (99.2, 63.0)
- added R19: RESISTORAXIAL-0.3, Resistors:AXIAL-0.3, F.Cu at (104.3, 72.3)
- added R20: RESISTORAXIAL-0.3, Resistors:AXIAL-0.3, F.Cu at (104.8, 92.4)
- added R21: RESISTORAXIAL-0.3, Resistors:AXIAL-0.3, F.Cu at (95.5, 88.4)
- added R22: RESISTORAXIAL-0.3, Resistors:AXIAL-0.3, F.Cu at (99.1, 72.3)
- moved R18 84.1 mm to (102.4, 132.0), turned to 0 degrees
- moved R17 78.0 mm to (102.5, 106.5), turned to 180 degrees
- moved J1 56.3 mm to (205.7, 63.1)
- moved J2 56.3 mm to (159.0, 63.1)
- moved U1 56.3 mm to (150.3, 130.1)
- moved R10 42.6 mm to (185.4, 55.9), turned to -90 degrees
- moved R13 42.4 mm to (128.5, 55.9), turned to -90 degrees
- moved R4 42.1 mm to (200.6, 55.9), turned to -90 degrees
- moved R3 42.0 mm to (190.5, 55.9), turned to -90 degrees
- moved R5 42.0 mm to (123.4, 55.9), turned to -90 degrees
- moved R12 42.0 mm to (205.7, 55.9), turned to -90 degrees
- moved R11 42.0 mm to (195.5, 55.9), turned to -90 degrees
- moved R1 41.9 mm to (170.2, 55.9), turned to -90 degrees
- moved R7 41.9 mm to (143.7, 55.9), turned to -90 degrees
- moved R2 41.9 mm to (180.3, 55.9), turned to -90 degrees
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Connections:
- U1 pad 23: /ct10 -> /ct9
- U1 pad 24: /ct11 -> /ct10
- U1 pad 30: /ct8 -> Net-(U1-Pad30)
- U1 pad 32: /ct12 -> /ct11
- U1 pad 33: /ct13 -> /ct12
- U1 pad 34: /ct14 -> /ct13
- U1 pad 35: /ct15 -> /ct14
- U1 pad 36: /ct16 -> /ct15
- U1 pad 38: Net-(U1-Pad38) -> /ct16
- U1 pad 43: /ct9 -> /ct3
- U1 pad 44: /ct3 -> /ct4
- U1 pad 45: /ct4 -> /ct5
- U1 pad 46: /ct5 -> /ct6
- U1 pad 47: /ct6 -> /ct7
- U1 pad 48: Net-(U1-Pad48) -> Net-(R21-PadP$2)
- U1 pad 49: Net-(U1-Pad49) -> Net-(R19-PadP$2)
- U1 pad 50: /ct7 -> /ct8
- U1 pad 56: Net-(U1-Pad56) -> Net-(R19-PadP$2)
- U1 pad 57: Net-(U1-Pad57) -> Net-(R21-PadP$2)
Routing:
- net /CT_BIAS: track 115.6 -> 391.6 mm
- net /ct9: track 0.00 -> 102.3 mm
- net Net-(R21-PadP$2): track 0.00 -> 100.4 mm
- net /ct10: track 0.00 -> 87.4 mm
- net Net-(R19-PadP$2): track 0.00 -> 85.1 mm
- net /ct11: track 0.00 -> 71.7 mm
- net /ct12: track 0.00 -> 70.6 mm
- net /ct13: track 0.00 -> 70.0 mm
- net /ct14: track 0.00 -> 68.5 mm
- net /ct16: track 0.00 -> 67.7 mm
- net /ct15: track 0.00 -> 67.4 mm
- net /ct1: track 0.00 -> 66.5 mm
- net /ct7: track 0.00 -> 66.2 mm
- net /ct2: track 0.00 -> 65.4 mm
- net /ct8: track 0.00 -> 65.2 mm
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
Commit message: good looking board now
Parts:
- moved R10 42.4 mm to (179.1, 97.8)
- moved R12 42.4 mm to (199.4, 97.8)
- moved R2 42.4 mm to (174.0, 97.8)
- moved R3 42.4 mm to (184.2, 97.8)
- moved R4 42.4 mm to (194.3, 97.8)
- moved R9 42.4 mm to (168.9, 97.8)
- moved R1 42.4 mm to (163.8, 97.8)
- moved R11 42.4 mm to (189.2, 97.8)
- moved R13 42.0 mm to (125.7, 97.8)
- moved R14 42.0 mm to (135.9, 97.8)
- moved R15 42.0 mm to (146.1, 97.8)
- moved R16 42.0 mm to (156.2, 97.8)
- moved R5 42.0 mm to (120.7, 97.8)
- moved R6 42.0 mm to (130.8, 97.8)
- moved R7 42.0 mm to (141.0, 97.8)
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Connections:
- U1 pad 1: Net-(U1-Pad1) -> /GND
- U1 pad 15: Net-(U1-Pad15) -> /3.3V
- U1 pad 39: /GND -> Net-(U1-Pad39)
- U1 pad 51: /3.3V -> Net-(U1-Pad51)
Routing:
- net /CT_BIAS: track 391.6 -> 219.3 mm
- net Net-(R21-PadP$2): track 100.4 -> 42.5 mm
- net /ct9: track 102.3 -> 49.5 mm
- net Net-(R19-PadP$2): track 85.1 -> 32.8 mm
- net /3.3V: track 26.4 -> 74.5 mm
- net /ct10: track 87.4 -> 40.1 mm
- net /ct13: track 70.0 -> 22.7 mm
- net /ct16: track 67.7 -> 20.6 mm
- net /ct14: track 68.5 -> 21.7 mm
- net /ct15: track 67.4 -> 20.6 mm
- net /ct1: track 66.5 -> 20.7 mm
- net /ct12: track 70.6 -> 25.0 mm
- net /ct2: track 65.4 -> 20.6 mm
- net /ct11: track 71.7 -> 27.2 mm
- net /ct3: track 63.8 -> 21.7 mm
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Other:
- board outline added: 118.1 x 53.3 mm

Commit message: sch and pcb look good, also gbr and ngc outputs
Connections:
- net Net-(R19-PadP$2) renamed /L2_SCALED
- net Net-(R21-PadP$2) renamed /L1_SCALED
Other:
- board size 118.1 x 53.3 mm -> 146.1 x 78.7 mm
