File: hardware/teensy/teensy.kicad_pcb (KiCad board)
At the start: 2 copper layers, 146.1 x 78.7 mm, 26 parts, among them J1 CONN_16, J2 CONN_16, J3 CONN_04, U1 Teensy3.5

Commit message: hoo boy, adc protection and bigger terminals
Parts:
- added RV1: R_POT_US, Potentiometer_THT:Potentiometer_Bourns_3296W_Vertical, F.Cu at (163.8, 82.5)
- J1, J2: value CONN_16 -> ~
- J3: value CONN_04 -> ~
- R1, R10, R11, R12, R13, R14, R15, R16, R17, R18, R19, R2, R20, R21, R22, R3, R4, R5, R6, R7, R8, R9: value RESISTORAXIAL-0.3 -> ~
- U1: value Teensy3.5 -> ~
Connections:
- R1 pad P$1: /CT_BIAS -> Net-(R1-PadP$1)

Commit message: layout
Parts:
- removed J1, J2: ~, Connectors:1X16
- removed J3: ~, Connectors:1X04
- added D1: D_Schottky, Diode_SMD:D_SOD-123, B.Cu at (224.8, 94.0)
- added D10: D_Schottky, Diode_SMD:D_SOD-123, B.Cu at (172.7, 135.9)
- added D11: D_Schottky, Diode_SMD:D_SOD-123, B.Cu at (186.7, 94.0)
- added D12: D_Schottky, Diode_SMD:D_SOD-123, B.Cu at (162.6, 135.9)
- added D13: D_Schottky, Diode_SMD:D_SOD-123, B.Cu at (179.1, 94.0)
- added D14: D_Schottky, Diode_SMD:D_SOD-123, B.Cu at (160.0, 135.9)
- added D15: D_Schottky, Diode_SMD:D_SOD-123, B.Cu at (171.4, 94.0)
- added D16: D_Schottky, Diode_SMD:D_SOD-123, B.Cu at (157.5, 135.9)
- added D17: D_Schottky, Diode_SMD:D_SOD-123, B.Cu at (163.8, 94.0)
- added D18: D_Schottky, Diode_SMD:D_SOD-123, B.Cu at (154.9, 135.9)
- added D19: D_Schottky, Diode_SMD:D_SOD-123, B.Cu at (156.2, 94.0)
- added D2: D_Schottky, Diode_SMD:D_SOD-123, B.Cu at (180.3, 138.4)
- added D20: D_Schottky, Diode_SMD:D_SOD-123, B.Cu at (152.4, 135.9)
- added D21: D_Schottky, Diode_SMD:D_SOD-123, B.Cu at (148.6, 94.0)
- added D22: D_Schottky, Diode_SMD:D_SOD-123, B.Cu at (149.9, 135.9)
- added D23: D_Schottky, Diode_SMD:D_SOD-123, B.Cu at (141.0, 94.0)
- added D24: D_Schottky, Diode_SMD:D_SOD-123, B.Cu at (147.3, 135.9)
- added D25: D_Schottky, Diode_SMD:D_SOD-123, B.Cu at (110.5, 94.0)
- added D26: D_Schottky, Diode_SMD:D_SOD-123, B.Cu at (129.5, 135.9)
- added D27: D_Schottky, Diode_SMD:D_SOD-123, B.Cu at (118.1, 94.0)
- added D28: D_Schottky, Diode_SMD:D_SOD-123, B.Cu at (139.7, 135.9)
- added D29: D_Schottky, Diode_SMD:D_SOD-123, B.Cu at (125.7, 94.0)
- added D3: D_Schottky, Diode_SMD:D_SOD-123, B.Cu at (217.2, 94.0)
- added D30: D_Schottky, Diode_SMD:D_SOD-123, B.Cu at (142.2, 135.9)
- added D31: D_Schottky, Diode_SMD:D_SOD-123, B.Cu at (133.3, 94.0)
- added D32: D_Schottky, Diode_SMD:D_SOD-123, B.Cu at (144.8, 135.9)
- added D33: D_Schottky, Diode_SMD:D_SOD-123, B.Cu at (68.6, 81.3)
- added D34: D_Schottky, Diode_SMD:D_SOD-123, B.Cu at (134.6, 135.9)
- added D35: D_Schottky, Diode_SMD:D_SOD-123, B.Cu at (58.4, 81.3)
- added D36: D_Schottky, Diode_SMD:D_SOD-123, B.Cu at (137.2, 135.9)
- added D4: D_Schottky, Diode_SMD:D_SOD-123, B.Cu at (182.9, 138.4)
- added D5: D_Schottky, Diode_SMD:D_SOD-123, B.Cu at (209.6, 94.0)
- added D6: D_Schottky, Diode_SMD:D_SOD-123, B.Cu at (177.8, 135.9)
- added D7: D_Schottky, Diode_SMD:D_SOD-123, B.Cu at (201.9, 94.0)
- added D8: D_Schottky, Diode_SMD:D_SOD-123, B.Cu at (175.3, 135.9)
- added D9: D_Schottky, Diode_SMD:D_SOD-123, B.Cu at (194.3, 94.0)
- added J4: CONN_083.5MM-8, Connectors:SCREWTERMINAL-3.5MM-8, F.Cu at (190.5, 31.8)
- added J5: CONN_083.5MM-8, Connectors:SCREWTERMINAL-3.5MM-8, F.Cu at (221.0, 31.8)
- added J6: CONN_083.5MM-8, Connectors:SCREWTERMINAL-3.5MM-8, F.Cu at (129.5, 31.8)
- added J7: CONN_083.5MM-8, Connectors:SCREWTERMINAL-3.5MM-8, F.Cu at (160.0, 31.8)
- added J8: CONN_023.5MM, Connectors:SCREWTERMINAL-3.5MM-2, F.Cu at (62.2, 31.8)
- added J9: CONN_023.5MM, Connectors:SCREWTERMINAL-3.5MM-2, F.Cu at (53.3, 31.8)
- added R23: ~, Resistors:AXIAL-0.3, F.Cu at (221.0, 91.4)
- added R24: ~, Resistors:AXIAL-0.3, F.Cu at (213.4, 91.4)
- added R25: ~, Resistors:AXIAL-0.3, F.Cu at (205.7, 91.4)
- added R26: ~, Resistors:AXIAL-0.3, F.Cu at (198.1, 91.4)
- added R27: ~, Resistors:AXIAL-0.3, F.Cu at (190.5, 91.4)
- added R28: ~, Resistors:AXIAL-0.3, F.Cu at (182.9, 91.4)
- added R29: ~, Resistors:AXIAL-0.3, F.Cu at (175.3, 91.4)
- added R30: ~, Resistors:AXIAL-0.3, F.Cu at (167.6, 91.4)
- added R31: ~, Resistors:AXIAL-0.3, F.Cu at (160.0, 91.4)
- added R32: ~, Resistors:AXIAL-0.3, F.Cu at (152.4, 91.4)
- added R33: ~, Resistors:AXIAL-0.3, F.Cu at (144.8, 91.4)
- added R34: ~, Resistors:AXIAL-0.3, F.Cu at (137.2, 91.4)
- added R35: ~, Resistors:AXIAL-0.3, F.Cu at (106.7, 91.4)
- added R36: ~, Resistors:AXIAL-0.3, F.Cu at (114.3, 91.4)
- added R37: ~, Resistors:AXIAL-0.3, F.Cu at (121.9, 91.4)
- added R38: ~, Resistors:AXIAL-0.3, F.Cu at (129.5, 91.4)
- added RV10: R_POT_US, Potentiometer_THT:Potentiometer_Bourns_3296W_Vertical, F.Cu at (114.3, 62.2)
- added RV11: R_POT_US, Potentiometer_THT:Potentiometer_Bourns_3296W_Vertical, F.Cu at (121.9, 62.2)
- added RV12: R_POT_US, Potentiometer_THT:Potentiometer_Bourns_3296W_Vertical, F.Cu at (129.5, 62.2)
- added RV13: R_POT_US, Potentiometer_THT:Potentiometer_Bourns_3296W_Vertical, F.Cu at (137.2, 62.2)
- added RV14: R_POT_US, Potentiometer_THT:Potentiometer_Bourns_3296W_Vertical, F.Cu at (144.8, 62.2)
- added RV15: R_POT_US, Potentiometer_THT:Potentiometer_Bourns_3296W_Vertical, F.Cu at (152.4, 62.2)
- added RV16: R_POT_US, Potentiometer_THT:Potentiometer_Bourns_3296W_Vertical, F.Cu at (160.0, 62.2)
- added RV17: R_POT_US, Potentiometer_THT:Potentiometer_Bourns_3296W_Vertical, F.Cu at (64.8, 62.2)
- added RV18: R_POT_US, Potentiometer_THT:Potentiometer_Bourns_3296W_Vertical, F.Cu at (54.6, 62.2)
- added RV2: R_POT_US, Potentiometer_THT:Potentiometer_Bourns_3296W_Vertical, F.Cu at (175.3, 62.2)
- added RV3: R_POT_US, Potentiometer_THT:Potentiometer_Bourns_3296W_Vertical, F.Cu at (182.9, 62.2)
- added RV4: R_POT_US, Potentiometer_THT:Potentiometer_Bourns_3296W_Vertical, F.Cu at (190.5, 62.2)
- added RV5: R_POT_US, Potentiometer_THT:Potentiometer_Bourns_3296W_Vertical, F.Cu at (198.1, 62.2)
- added RV6: R_POT_US, Potentiometer_THT:Potentiometer_Bourns_3296W_Vertical, F.Cu at (205.7, 62.2)
- added RV7: R_POT_US, Potentiometer_THT:Potentiometer_Bourns_3296W_Vertical, F.Cu at (213.4, 62.2)
- added RV8: R_POT_US, Potentiometer_THT:Potentiometer_Bourns_3296W_Vertical, F.Cu at (221.0, 62.2)
- added RV9: R_POT_US, Potentiometer_THT:Potentiometer_Bourns_3296W_Vertical, F.Cu at (106.7, 62.2)
- moved R17 68.6 mm to (29.2, 95.2)
- moved R18 68.6 mm to (34.3, 95.2)
- moved R22 59.0 mm to (52.1, 78.7)
- moved R21 59.0 mm to (54.6, 78.7)
- moved R19 54.3 mm to (62.2, 78.7)
- moved R20 54.3 mm to (64.8, 78.7)
- moved R12 28.8 mm to (221.0, 78.7)
- moved R4 26.9 mm to (213.4, 78.7)
- moved R11 25.2 mm to (205.7, 78.7)
- moved R3 23.6 mm to (198.1, 78.7)
- moved R5 23.6 mm to (106.7, 78.7)
- moved R10 22.2 mm to (190.5, 78.7)
- moved R13 22.2 mm to (114.3, 78.7)
- moved R6 21.0 mm to (121.9, 78.7)
- moved R2 21.0 mm to (182.9, 78.7)
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Connections:
- R10 pad P$1: /CT_BIAS -> Net-(R10-PadP$1)
- R11 pad P$1: /CT_BIAS -> Net-(R11-PadP$1)
- R12 pad P$1: /CT_BIAS -> Net-(R12-PadP$1)
- R13 pad P$1: /CT_BIAS -> Net-(R13-PadP$1)
- R14 pad P$1: /CT_BIAS -> Net-(R14-PadP$1)
- R15 pad P$1: /CT_BIAS -> Net-(R15-PadP$1)
- R16 pad P$1: /CT_BIAS -> Net-(R16-PadP$1)
- R2 pad P$1: /CT_BIAS -> Net-(R2-PadP$1)
- R20 pad P$2: /CT_BIAS -> Net-(R20-PadP$2)
- R21 pad P$1: /CT_BIAS -> Net-(R21-PadP$1)
- R3 pad P$1: /CT_BIAS -> Net-(R3-PadP$1)
- R4 pad P$1: /CT_BIAS -> Net-(R4-PadP$1)
- R5 pad P$1: /CT_BIAS -> Net-(R5-PadP$1)
- R6 pad P$1: /CT_BIAS -> Net-(R6-PadP$1)
- R7 pad P$1: /CT_BIAS -> Net-(R7-PadP$1)
- R8 pad P$1: /CT_BIAS -> Net-(R8-PadP$1)
- R9 pad P$1: /CT_BIAS -> Net-(R9-PadP$1)
- U1 pad 23: /ct9 -> Net-(D1-Pad1)
- U1 pad 24: /ct10 -> Net-(D3-Pad1)
- U1 pad 32: /ct11 -> Net-(D5-Pad1)
- U1 pad 33: /ct12 -> Net-(D7-Pad1)
- U1 pad 34: /ct13 -> Net-(D10-Pad2)
- U1 pad 35: /ct14 -> Net-(D11-Pad1)
- U1 pad 36: /ct15 -> Net-(D13-Pad1)
- U1 pad 38: /ct16 -> Net-(D15-Pad1)
- U1 pad 41: /ct1 -> Net-(D17-Pad1)
- U1 pad 42: /ct2 -> Net-(D19-Pad1)
- U1 pad 43: /ct3 -> Net-(D21-Pad1)
- U1 pad 44: /ct4 -> Net-(D23-Pad1)
- U1 pad 45: /ct5 -> Net-(D31-Pad1)
- U1 pad 46: /ct6 -> Net-(D29-Pad1)
- U1 pad 47: /ct7 -> Net-(D27-Pad1)
- U1 pad 50: /ct8 -> Net-(D25-Pad1)
Routing:
- net /CT_BIAS: track 219.3 -> 0.00 mm
- net /3.3V: track 74.5 -> 0.00 mm
- net /ct9: track 49.5 -> 0.00 mm
- net /L1_SCALED: track 42.5 -> 0.00 mm
- net /ct10: track 40.1 -> 0.00 mm
- net /L2_SCALED: track 32.8 -> 0.00 mm
- net /GND: track 31.8 -> 0.00 mm
- net /ct7: track 30.4 -> 0.00 mm
- net /ct8: track 28.1 -> 0.00 mm
- net /ct6: track 27.5 -> 0.00 mm
- net /ct11: track 27.2 -> 0.00 mm
- net /ct12: track 25.0 -> 0.00 mm
- net /ct5: track 25.0 -> 0.00 mm
- net /ct13: track 22.7 -> 0.00 mm
- net /ct4: track 22.7 -> 0.00 mm
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
Commit message: prettier traces, removed smt thing
Parts:
- U1: footprint teensy:Teensy35_36 -> teensy:Teensy35_36_EMON
- moved R17 42.1 mm to (71.2, 91.4)
- moved R18 42.1 mm to (76.2, 91.4)
- moved J8 39.7 mm to (95.5, 53.3)
- moved J9 36.6 mm to (82.9, 53.3)
- moved D33 36.6 mm to (102.9, 94.0)
- moved R20 36.6 mm to (99.1, 91.4)
- moved RV17 34.3 mm to (99.1, 62.2)
- moved R19 34.2 mm to (94.0, 91.4)
- moved D35 34.2 mm to (90.2, 94.0)
- moved R21 34.2 mm to (86.4, 91.4)
- moved R22 31.9 mm to (81.3, 91.4)
- moved RV18 31.8 mm to (86.4, 62.2)
- moved J4 21.9 mm to (194.3, 53.3)
- moved J5 21.9 mm to (224.8, 53.3)
- moved J6 21.9 mm to (133.3, 53.3)
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Connections:
- net /L1_SCALED renamed /A11_A7
- net /L2_SCALED renamed /A10_A8
- net Net-(D1-Pad1) renamed /A12
- net Net-(D10-Pad2) renamed /A18
- net Net-(D11-Pad1) renamed /A19
- net Net-(D13-Pad1) renamed /A20
- net Net-(D15-Pad1) renamed /A22
- net Net-(D17-Pad1) renamed /A0
- net Net-(D19-Pad1) renamed /A1
- net Net-(D21-Pad1) renamed /A2
- net Net-(D23-Pad1) renamed /A3
- net Net-(D25-Pad1) renamed /A9
- net Net-(D27-Pad1) renamed /A6
- net Net-(D29-Pad1) renamed /A5
- net Net-(D3-Pad1) renamed /A13
- net Net-(D31-Pad1) renamed /A4
- net Net-(D5-Pad1) renamed /A16
- net Net-(D7-Pad1) renamed /A17
- D26 pad 1: /3.3V -> /3.3V_2
- D34 pad 1: /3.3V -> /3.3V_2
- U1 pad 51: Net-(U1-Pad51) -> /3.3V_2
Routing:
- net /CT_BIAS: track 0.00 -> 288.4 mm
- net /GND: track 0.00 -> 243.1 mm
- net /3.3V: track 0.00 -> 143.1 mm
- net /A11_A7: track 0.00 -> 94.0 mm
- net /A12: track 0.00 -> 82.5 mm
- net /A10_A8: track 0.00 -> 75.8 mm
- net /A13: track 0.00 -> 69.6 mm
- net /A6: track 0.00 -> 56.4 mm
- net /A16: track 0.00 -> 54.5 mm
- net /A5: track 0.00 -> 54.3 mm
- net /A17: track 0.00 -> 52.4 mm
- net /A4: track 0.00 -> 52.2 mm
- net /A9: track 0.00 -> 51.5 mm
- net /A3: track 0.00 -> 50.4 mm
- net /A18: track 0.00 -> 50.3 mm
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Other:
- board size 146.1 x 78.7 mm -> 254 x 190.5 mm

Commit message: a little more beauty
Routing:
- net /CT_BIAS: track 288.4 -> 445.6 mm
- net /ct4: track 29.5 -> 35.5 mm
- net /3.3V: track 143.1 -> 138.7 mm
- net /ct2: track 36.1 -> 34.7 mm
- net /ct12: track 36.6 -> 35.5 mm
- net /ct16: track 36.6 -> 35.5 mm
- net /ct8: track 36.6 -> 35.5 mm
- net /ct7: track 36.4 -> 35.4 mm
- net /ct3: track 36.4 -> 35.4 mm
- net /ct11: track 36.4 -> 35.4 mm
- net /ct15: track 36.4 -> 35.4 mm
- net /A3: track 50.4 -> 49.5 mm
- net /ct10: track 36.1 -> 35.4 mm
- net /ct6: track 36.1 -> 35.4 mm
- net /ct14: track 36.1 -> 35.4 mm
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
Commit message: updated gbr and ngc
Routing:
- net /L1: track 34.9 -> 34.4 mm
- net /L2: track 34.9 -> 34.4 mm
Other:
- board size 254 x 190.5 mm -> 215.9 x 152.4 mm
Changed lines of the file:
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@@
     )
     (pcbplotparams
-      (layerselection 0x010fc_ffffffff)
+      (layerselection 0x01000_fffffffe)
       (usegerberextensions false)
       (usegerberattributes false)
@@
     )
   )
-  (gr_rect (start 12.7 12.7) (end 266.7 203.2) (layer "Edge.Cuts") (width 0.1))
+  (gr_rect (start 38.1 25.4) (end 254 177.8) (layer "Edge.Cuts") (width 0.1))
+  (segment (start 82.86242 53.34) (end 81.28 62.23) (width 1.778) (layer "B.Cu") (net 45))
+  (segment (start 81.28 62.23) (end 81.28 87.602466) (width 1.778) (layer "B.Cu") (net 45))
+  (segment (start 95.547343 53.34) (end 93.98 62.23) (width 1.778) (layer "B.Cu") (net 48))
+  (segment (start 93.98 62.23) (end 93.98 87.63) (width 1.778) (layer "B.Cu") (net 48))
   (segment (start 122.85218 53.34) (end 121.92 62.23) (width 1.778) (layer "B.Cu") (net 43))
   (segment (start 115.85194 51.90316) (end 116.980501 50.774599) (width 1.778) (layer "B.Cu") (net 43))
@@
   (segment (start 93.98 95.25) (end 99.06 95.25) (width 1.905) (layer "B.Cu") (net 84))
   (segment (start 106.68 96.52) (end 132.08 121.92) (width 1.778) (layer "B.Cu") (net 80))
-  (segment (start 106.68 95.25) (end 106.68 96.52) (width 0.762) (layer "B.Cu") (net 80))
+  (segment (start 106.68 95.25) (end 106.68 96.52) (width 1.778) (layer "B.Cu") (net 80))
   (segment (start 132.08 121.92) (end 132.08 123.19) (width 1.778) (layer "B.Cu") (net 80))
   (segment (start 114.3 96.52) (end 139.7 121.92) (width 1.778) (layer "B.Cu") (net 81))
-  (segment (start 114.3 95.25) (end 114.3 96.52) (width 0.762) (layer "B.Cu") (net 81))
+  (segment (start 114.3 95.25) (end 114.3 96.52) (width 1.778) (layer "B.Cu") (net 81))
   (segment (start 139.7 121.92) (end 139.7 129.54) (width 1.778) (layer "B.Cu") (net 81))
   (segment (start 121.92 96.36125) (end 142.24 116.68125) (width 1.778) (layer "B.Cu") (net 82))
-  (segment (start 121.92 95.25) (end 121.92 96.36125) (width 0.762) (layer "B.Cu") (net 82))
+  (segment (start 121.92 95.25) (end 121.92 96.36125) (width 1.778) (layer "B.Cu") (net 82))
   (segment (start 142.24 116.68125) (end 142.24 129.54) (width 1.778) (layer "B.Cu") (net 82))
   (segment (start 129.54 96.52) (end 144.78 111.76) (width 1.778) (layer "B.Cu") (net 83))
-  (segment (start 129.54 95.25) (end 129.54 96.52) (width 0.762) (layer "B.Cu") (net 83))
+  (segment (start 129.54 95.25) (end 129.54 96.52) (width 1.778) (layer "B.Cu") (net 83))
   (segment (start 144.78 111.76) (end 144.78 129.54) (width 1.778) (layer "B.Cu") (net 83))
   (segment (start 137.16 96.52) (end 147.32 106.68) (width 1.778) (layer "B.Cu") (net 79))
-  (segment (start 137.16 95.25) (end 137.16 96.52) (width 0.762) (layer "B.Cu") (net 79))
+  (segment (start 137.16 95.25) (end 137.16 96.52) (width 1.778) (layer "B.Cu") (net 79))
   (segment (start 147.32 106.68) (end 147.32 129.54) (width 1.778) (layer "B.Cu") (net 79))
   (segment (start 182.88 96.52) (end 170.18 109.22) (width 1.778) (layer "B.Cu") (net 73))
-  (segment (start 182.88 95.25) (end 182.88 96.52) (width 0.762) (layer "B.Cu") (net 73))
+  (segment (start 182.88 95.25) (end 182.88 96.52) (width 1.778) (layer "B.Cu") (net 73))
   (segment (start 170.18 109.22) (end 170.18 129.54) (width 1.778) (layer "B.Cu") (net 73))
   (segment (start 190.5 96.52) (end 172.72 114.3) (width 1.778) (layer "B.Cu") (net 72))
-  (segment (start 190.5 95.25) (end 190.5 96.52) (width 0.762) (layer "B.Cu") (net 72))
+  (segment (start 190.5 95.25) (end 190.5 96.52) (width 1.778) (layer "B.Cu") (net 72))
   (segment (start 172.72 114.3) (end 172.72 129.54) (width 1.778) (layer "B.Cu") (net 72))
   (segment (start 198.12 96.52) (end 175.26 119.38) (width 1.778) (layer "B.Cu") (net 71))
-  (segment (start 175.26 119.38) (end 175.26 129.54) (width 1.905) (layer "B.Cu") (net 71))
-  (segment (start 198.12 95.25) (end 198.12 96.52) (width 0.762) (layer "B.Cu") (net 71))
+  (segment (start 175.26 119.38) (end 175.26 129.54) (width 1.778) (layer "B.Cu") (net 71))
+  (segment (start 198.12 95.25) (end 198.12 96.52) (width 1.778) (layer "B.Cu") (net 71))
   (segment (start 205.74 96.52) (end 177.8 124.46) (width 1.778) (layer "B.Cu") (net 70))
-  (segment (start 205.74 95.25) (end 205.74 96.52) (width 0.762) (layer "B.Cu") (net 70))
+  (segment (start 205.74 95.25) (end 205.74 96.52) (width 1.778) (layer "B.Cu") (net 70))
   (segment (start 177.8 124.46) (end 177.8 129.54) (width 1.778) (layer "B.Cu") (net 70))
   (segment (start 167.64 96.36125) (end 162.56 101.44125) (width 1.778) (layer "B.Cu") (net 75))
-  (segment (start 167.64 95.25) (end 167.64 96.36125) (width 0.762) (layer "B.Cu") (net 75))
+  (segment (start 167.64 95.25) (end 167.64 96.36125) (width 1.778) (layer "B.Cu") (net 75))
   (segment (start 162.56 101.44125) (end 162.56 129.54) (width 1.778) (layer "B.Cu") (net 75))
   (segment (start 175.26 96.52) (end 167.64 104.14) (width 1.778) (layer "B.Cu") (net 74))
-  (segment (start 175.26 95.25) (end 175.26 96.52) (width 0.762) (layer "B.Cu") (net 74))
+  (segment (start 175.26 95.25) (end 175.26 96.52) (width 1.778) (layer "B.Cu") (net 74))
   (segment (start 167.64 104.14) (end 167.64 129.54) (width 1.778) (layer "B.Cu") (net 74))
   (segment (start 149.86 101.6) (end 144.78 96.52) (width 1.778) (layer "B.Cu") (net 78))
   (segment (start 149.86 129.54) (end 149.86 101.6) (width 1.778) (layer "B.Cu") (net 78))
-  (segment (start 144.78 96.52) (end 144.78 95.25) (width 0.762) (layer "B.Cu") (net 78))
+  (segment (start 144.78 96.52) (end 144.78 95.25) (width 1.778) (layer "B.Cu") (net 78))
   (segment (start 154.94 101.6) (end 160.02 96.52) (width 1.778) (layer "B.Cu") (net 76))
   (segment (start 154.94 129.54) (end 154.94 101.6) (width 1.778) (layer "B.Cu") (net 76))
-  (segment (start 160.02 96.52) (end 160.02 95.25) (width 0.762) (layer "B.Cu") (net 76))
+  (segment (start 160.02 96.52) (end 160.02 95.25) (width 1.778) (layer "B.Cu") (net 76))
   (segment (start 76.2 53.34) (end 76.241012 87.63) (width 1.778) (layer "B.Cu") (net 43))
   (segment (start 99.044923 53.34) (end 108.8517 53.34) (width 1.778) (layer "B.Cu") (net 43))
@@
   (segment (start 99.06 62.23) (end 99.06 53.355077) (width 1.778) (layer "B.Cu") (net 43))
   (segment (start 129.54 62.23) (end 129.54 53.65242) (width 1.778) (layer "B.Cu") (net 43))
-  (segment (start 95.547343 53.34) (end 93.98 54.907343) (width 1.778) (layer "B.Cu") (net 48))
-  (segment (start 93.98 54.907343) (end 93.98 87.63) (width 1.778) (layer "B.Cu") (net 48))
-  (segment (start 81.28 54.92242) (end 81.28 87.602466) (width 1.778) (layer "B.Cu") (net 45))
-  (segment (start 82.86242 53.34) (end 81.28 54.92242) (width 1.778) (layer "B.Cu") (net 45))
   (segment (start 129.54 129.54) (end 129.54 126.11) (width 0.762) (layer "B.Cu") (net 67))
   (segment (start 120.65 126.62) (end 129.03 126.62) (width 0.762) (layer "B.Cu") (net 67))
@@
   (segment (start 109.22 144.78) (end 67.041478 102.601478) (width 1.778) (layer "B.Cu") (net 47))
   (segment (start 73.66 92.71) (end 76.2 95.25) (width 1.778) (layer "B.Cu") (net 47))
-  (segment (start 124.46 144.78) (end 109.22 144.78) (width 1.905) (layer "B.Cu") (net 47))
+  (segment (start 124.46 144.78) (end 109.22 144.78) (width 1.778) (layer "B.Cu") (net 47))
   (segment (start 67.041478 102.601478) (end 67.041478 95.518522) (width 1.778) (layer "B.Cu") (net 47))
   (segment (start 67.041478 95.518522) (end 69.85 92.71) (width 1.778) (layer "B.Cu") (net 47))
   (segment (start 69.85 92.71) (end 73.66 92.71) (width 1.778) (layer "B.Cu") (net 47))
   (segment (start 86.36 106.68) (end 116.380521 136.700521) (width 1.778) (layer "B.Cu") (net 85))
-  (segment (start 116.380521 136.700521) (end 133.670849 136.700521) (width 1.905) (layer "B.Cu") (net 85))
+  (segment (start 116.380521 136.700521) (end 133.670849 136.700521) (width 1.778) (layer "B.Cu") (net 85))
   (segment (start 86.36 95.25) (end 86.36 106.68) (width 1.778) (layer "B.Cu") (net 85))
   (segment (start 133.670849 136.700521) (end 137.16 133.21137) (width 1.778) (layer "B.Cu") (net 85))
-  (segment (start 137.16 133.21137) (end 137.16 132.08) (width 0.762) (layer "B.Cu") (net 85))
+  (segment (start 137.16 133.21137) (end 137.16 132.08) (width 1.778) (layer "B.Cu") (net 85))
   (segment (start 90.17 92.33) (end 79.161012 92.33) (width 0.762) (layer "B.Cu") (net 47))
   (segment (start 79.161012 92.33) (end 76.241012 95.25) (width 0.762) (layer "B.Cu") (net 47))
@@
   (segment (start 175.26 82.55) (end 175.26 87.63) (width 1.905) (layer "B.Cu") (net 26))
   (segment (start 182.88 82.55) (end 182.88 87.63) (width 1.905) (layer "B.Cu") (net 27))
-  (segment (start 190.5 82.55) (end 190.5 87.63) (width 0.762) (layer "B.Cu") (net 28))
-  (segment (start 198.12 82.55) (end 198.12 87.63) (width 0.762) (layer "B.Cu") (net 29))
+  (segment (start 190.5 82.55) (end 190.5 87.63) (width 1.778) (layer "B.Cu") (net 28))
+  (segment (start 198.12 82.55) (end 198.12 87.63) (width 1.778) (layer "B.Cu") (net 29))
   (segment (start 205.74 82.55) (end 205.74 87.63) (width 1.778) (layer "B.Cu") (net 30))
   (segment (start 213.36 82.55) (end 213.36 87.63) (width 1.778) (layer "B.Cu") (net 31))
